File: SensorenPCB.kicad_sch (KiCad schematic)
At the start: 12 parts, among them IC1 VL53L1CXV0FY_1, IC2 VL53L1CXV0FY_1, J1 Conn_01x16_Socket, J2 EDT_SE-Shield_027, J3 Conn_01x16_Socket

Commit message: Schaltplan vervollständigt: I2C3/I2C4, LSM6DSO, Pull-ups, +5V global
Co-Authored-By: Claude Sonnet 5.5 <noreply@anthropic.com>
Claude-Session: https://claude.ai/code/session_01RKYw2izZ8h2aW2LrU4XKsk
Parts:
- added C5, C6: 100nF, Capacitor_SMD:C_0603_1608Metric_Pad1.08x0.95mm_HandSolder, symbol Device:C
- added R3, R4: 4.7k, Resistor_SMD:R_0603_1608Metric_Pad0.98x0.95mm_HandSolder, symbol Device:R
- added R5, R6, R7, R8: 10k, Resistor_SMD:R_0603_1608Metric_Pad0.98x0.95mm_HandSolder, symbol Device:R
- R1, R2: value 10k -> 4.7k
Connections:
- net +3V3: now also AC1.11 (SDO_AUX_), AC1.12 (CS), AC1.5 (VDDIO), AC1.8 (VDD), R1.1, R2.1, C5.1, C6.1, R3.1, R4.1, R5.1, R6.1, R7.1, R8.1
- net GND: now also AC1.1 (SDO/SA0), AC1.2 (SDX), AC1.3 (SCX), C5.2, C6.2
- net I2C3_INT: now also IC1.7 (GPIO1), R6.2
- net I2C3_RST: now also IC1.5 (XSHUT), R5.2
- net I2C3_SCL: now also AC1.13 (SCL), IC1.10 (SCL), R2.2
- net I2C3_SDA: now also AC1.14 (SDA), IC1.9 (SDA), R1.2
- net I2C4_INT: now also IC2.7 (GPIO1), R8.2
- net I2C4_RST: now also IC2.5 (XSHUT), R7.2
- net I2C4_SCL: now also IC2.10 (SCL), R4.2
- net I2C4_SDA: now also IC2.9 (SDA), R3.2
- net USART6_CTS: now also AC1.9 (INT2)
- net USART6_RTS: now also AC1.4 (INT1_)
- no-connect marks 2 -> 3
